File: PCB/Elspark/Elspark v6.brd (EAGLE design)
At the start: 60 x 50.5 mm, 43 parts, among them IC2 TLC274D, Q2 IRF540, Q5 BD139

Commit message: New PCB
Parts:
- removed +5V, GND, HALSENSOR: (no value), wirepad:2,15/1,0
- removed D1, D2: 1N4148DO35-7, diode:DO35-7
- removed R6: 1k5, rcl:0207/2V
- removed R7: 1k, rcl:0207/2V
- removed R8: k470, pot:CA6V
- added SV1: (no value), con-lstb:MA03-1
- added VCC_GND_TX_RX: (no value), con-lstb:MA04-1
- R1: value 1k -> 100; device rcl:0207/2V -> rcl:0204/7
- R18: device rcl:0207/2V -> rcl:0204/7
- R2: value 1k -> 1k8; device rcl:0207/2V -> rcl:0204/7
- R22: device rcl:0204/7 -> rcl:0207/2V
- moved R2 34.7 mm to (5.08, -7.62), turned to 0 degrees
- moved C7 34.2 mm to (33.0, 7.62), turned to 90 degrees
- moved R1 30.7 mm to (5.08, -3.81), turned to 0 degrees
- moved C10 28.2 mm to (25.4, 40.6)
- moved C4 25.7 mm to (30.5, 30.5), turned to 180 degrees
- moved R4 25.4 mm to (22.9, 48.9)
- moved R18 25.0 mm to (30.5, 26.7)
- moved R12 18.8 mm to (38.1, 24.1)
- moved R13 18.8 mm to (41.3, 24.1)
- moved B- 14.2 mm to (36.8, 14.6)
- moved C2 10.5 mm to (35.6, 41.9), turned to 90 degrees
- moved D5 9.16 mm to (48.3, 41.9), turned to 0 degrees
- moved R22 5.24 mm to (31.1, 41.9), turned to 270 degrees
- moved C5 2.84 mm to (50.8, 47.0)
- moved MODUL1 2.54 mm to (11.4, 27.9)
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Connections:
- removed net N$1: D1.A, R2.2
- removed net N$36: IC2.1
- removed net N$4: IC2.3, R6.2, R7.1
- removed net N$7: D2.A, R6.1
- removed net N$8: R7.2, R8.S
- new net 12V-MEASURE: IC2.1, IC2.2
- new net CPURX: MODUL1.J1.2, VCC_GND_TX_RX.3
- new net CPUTX: MODUL1.J1.1, VCC_GND_TX_RX.4
- net +12V: now also R2.2
- net +5V: now also SV1.1, VCC_GND_TX_RX.1; no longer +5V.1, R1.1, R8.E
- net GND: now also R1.1, SV1.3, VCC_GND_TX_RX.2; no longer D2.C, GND.1
- net M+: no longer D1.C
- net N$17: now also SV1.2; no longer HALSENSOR.1
- net N$2: now also IC2.3; no longer IC2.2
Routing:
- net GND: track 236.3 -> 0.00 mm, vias 1 -> 0
- net VCC: track 128.5 -> 0.00 mm
- net +5V: track 87.4 -> 0.00 mm
- net +12V: track 72.4 -> 0.00 mm, vias 4 -> 0
- net B+: track 68.7 -> 0.00 mm, vias 2 -> 0
- net N$35: track 59.1 -> 0.00 mm, vias 1 -> 0
- net TEMP: track 45.8 -> 0.00 mm
- net N$10: track 38.5 -> 0.00 mm
- net M+: track 23.0 -> 0.00 mm
- net N$4: track 22.4 -> 0.00 mm
- net N$11: track 19.2 -> 0.00 mm
- net N$23: track 18.6 -> 0.00 mm
- net POT: track 17.7 -> 0.00 mm
- net N$2: track 15.8 -> 0.00 mm
- net N$34: track 15.1 -> 0.00 mm, vias 1 -> 0
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