File: PCB/Elspark/Elspark v6.sch (EAGLE design)
At the start: 47 parts, among them IC2 TLC274D, Q5 IRF540, U1 IR2103

Commit message: New Elspark v6 arduino board
Parts:
- removed A4, A5, A6, RX, TX: (no value), wirepad:1,6/0,9
- removed BAT, SHUNT, VIN: (no value), con-wago-500:W237-102
- removed C15: 24u, rcl:CPOL-EUE2.5-5
- removed C16: 100n, rcl:C-EU050-024X044
- removed C6: 100u, rcl:CPOL-EUE2.5-5
- removed D6: Switch0, wirepad:1,6/0,9
- removed D7: Switch1, wirepad:1,6/0,9
- removed D8: Switch2, wirepad:1,6/0,9
- removed D9: Switch3, wirepad:1,6/0,9
- removed H1, H2, H3, H4: MOUNT-HOLE3.2, holes:MOUNT-HOLE3.2
- removed R19: 47k, rcl:R-EU_0207/2V
- removed R23: 47, rcl:R-EU_0207/2V
- removed R24, R25, R26, R27: 1k, rcl:R-EU_0207/2V
- removed R28: 2k7, rcl:R-EU_0207/2V
- removed R29: 0, rcl:R-EU_0207/2V
- removed R30, R31: 33k, rcl:R-EU_0207/2V
- removed R35: 100, rcl:R-EU_0207/2V
- removed R9: 680, rcl:R-EU_0207/2V
- removed U1: IR2103, irf-2:IR2103
- added +, +5V, -, GND, HALSENSOR, POT: (no value), wirepad:2,15/1,0
- added B+, B+1, B-, M-: WIREPAD4,16O1,6, wirepad:WIREPAD4,16O1,6
- added C1: 1000u, rcl:CPOL-EUE7.5-16
- added C10: 24u, rcl:CPOL-EUE2.5-5
- added C3, C4: 100n, rcl:C-EU050-024X044
- added C5: 100u, rcl:CPOL-EUE2.5-5
- added D13: MUR810, diode:MUR810
- added D2: 1N4148DO35-7, diode:1N4148DO35-7
- added D5: 11v, diode:BZX55
- added Q2: IRF540, transistor-power:IRF540
- added R1, R2: 1k, rcl:R-EU_0207/2V
- added R11, R20: 47, rcl:R-EU_0207/2V
- added R13: 1k8, rcl:R-EU_0204/7
- added R16: 47k, rcl:R-EU_0207/2V
- added R3: 10, rcl:R-EU_0207/2V
- added R4: 100k, ptc-ntc:NTC640-9
- added SWITCH: (no value), wirepad:1,6/0,9
- C7: value 100u -> 100n; device rcl:CPOL-EUE2.5-5 -> rcl:C-EU050-024X044
- Q5: value IRF540 -> BD139; device transistor-power:IRF540 -> transistor-power:BD139
- R12: value 39k -> 100; device rcl:R-EU_0207/2V -> rcl:R-EU_0204/7
- R18: value 100k -> 4k7; device ptc-ntc:NTC640-9 -> rcl:R-EU_0207/2V
- R22: value 47 -> 4k7; device rcl:R-EU_0207/2V -> rcl:R-EU_0204/7
- R5: value 3k3 -> 2k2
- R6: value 33k -> 1k5
- R7: value 33k -> 1k
- R8: value 3k3 -> k470; device rcl:R-EU_0207/2V -> pot:TRIM_EU-CA6V
- U$1: value MIC4451 -> MIC4451SO-8; device mic4451:MIC4451 -> mic4451:MIC4451SO-8
Connections:
- removed net B-/SHUNT: BAT-1.KL, IC2B.+IN, R6.1, SHUNT-2.KL
- removed net CHARGEPWM: MODUL1.D3, U1.HIN
- removed net CHOPEDPOWER: Q5.S
- removed net INVOLTAGESIGNAL: IC2D.OUT, MODUL1.A3, R29.2
- removed net N$12: MODUL1.D7, R25.2
- removed net N$14: MODUL1.D8, R26.2
- removed net N$15: MODUL1.D9, R27.2
- removed net N$16: A5.P, MODUL1.A5
- removed net N$18: MODUL1.D0/RX, RX.P
- removed net N$19: C15.-, C16.2
- removed net N$20: R35.1, U1.HO
- removed net N$24: IC2A.+IN, R5.1, R6.2
- removed net N$27: IC2A.-IN, R7.2, R8.1
- removed net N$3: IC2D.+IN, R28.1, R30.2
- removed net N$39: IC2C.-IN, R21.1, R22.1, R23.2
- removed net N$46: IC2C.+IN, R18.2, R19.1
- removed net N$48: IC2D.-IN, R29.1, R31.2
- removed net N$5: A4.P, MODUL1.A4
- removed net N$54: D6.P, R24.1
- removed net N$55: D7.P, R25.1
- removed net N$56: D8.P, R26.1
- removed net N$57: D9.P, R27.1
- removed net N$6: MODUL1.D1/TX, TX.P
- removed net OUTCURRENTSIGNAL: IC2B.OUT, MODUL1.A1, R12.2
- removed net OUTVOLTAGESIGNAL: IC2A.OUT, MODUL1.A0, R8.2
- removed net TEMPSIGNAL: IC2C.OUT, MODUL1.A2, R21.2
- removed net V+: Q5.D, R30.1
- removed net VB: C7.+, D1.C, U1.VB
- new net B+MEASURE: IC2C.-IN, IC2C.OUT
- new net HALSENS-MEASURE: C4.1, R18.2
- new net M+: D1.C, D13.A, M-.P, Q2.D
- new net N$1: D1.A, R2.2
- new net N$23: IC2D.-IN, R11.1, R20.1, R21.2
- new net N$34: POT.P, R22.1
- new net N$35: IC2D.+IN, R16.1, R4.2
- new net N$36: IC2A.OUT
- new net N$41: Q5.C, R5.2, SWITCH.P
- new net N$9: Q2.G, R3.1
- new net POT: C2.1, R22.2
- new net PWM: U$1.IN
- new net PWM-HIGH: R3.2, U$1.OUT, U$1.OUT2
- new net TEMP: C3.1, IC2D.OUT, R11.2
- new net VCC: +.P, C10.+, C7.1, IC2P.V+
- net +12V: now also C5.+, Q5.E, U$1.VDD, U$1.VDD2; no longer C2.1, C6.+, D1.A, U1.VCC
- net +5V: now also +5V.P, MODUL1.+5V, R1.1, R16.2, R20.2, R8.E; no longer C15.+, C16.1, R19.2, R22.2
- net B+: now also B+.P, B+1.P, C1.+, D13.C, R13.2; no longer BAT-2.KL, R7.1
- net GND: now also -.P, B-.P, C1.-, C10.-, C3.2, C4.2, C5.-, C7.2, D2.C, D5.A, GND.P, IC2P.V-, Q2.S, R12.1, R21.1, R4.1, U$1.GND, U$1.GND2; no longer C6.-, R18.1, R23.1, R28.2, R31.1, R5.2, R9.1, SHUNT-1.KL, U1./LIN, U1.COM
- net N$10: now also IC2C.+IN, R12.2, R13.1; no longer VIN-1.KL
- net N$11: now also D5.C, Q5.B, R5.1; no longer IC2B.-IN, R12.1, R9.2
- net N$17: now also HALSENSOR.P, R18.1; no longer A6.P, MODUL1.A6
- net N$2: now also IC2A.-IN, R1.2, R2.1; no longer C7.-, U1.VS
- net N$4: now also IC2A.+IN, R6.2, R7.1; no longer Q5.G, R35.2
- net N$7: now also D2.A, R6.1; no longer VIN-2.KL
- net N$8: now also R7.2, R8.S; no longer MODUL1.D6, R24.2
Other:
- note added: "B+ measure 0-95V"
- note added: "MOSFET current sens"
- note added: "Pot Measure"
- note removed: "Out Voltage Measure 0-40"
- note removed: "in Voltage Measure 0-66v"
- moved on the sheet: C2, D1, IC2A, IC2B, IC2C, IC2D, MODUL1, R12, R21, R22, R5, R6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

Commit message: New PCB
Parts:
- removed +5V, GND, HALSENSOR: (no value), wirepad:2,15/1,0
- removed D1, D2: 1N4148DO35-7, diode:1N4148DO35-7
- removed R6: 1k5, rcl:R-EU_0207/2V
- removed R7: 1k, rcl:R-EU_0207/2V
- removed R8: k470, pot:TRIM_EU-CA6V
- added SV1: (no value), con-lstb:MA03-1
- added VCC_GND_TX_RX: (no value), con-lstb:MA04-1
- R1: value 1k -> 100; device rcl:R-EU_0207/2V -> rcl:R-EU_0204/7
- R18: device rcl:R-EU_0207/2V -> rcl:R-EU_0204/7
- R2: value 1k -> 1k8; device rcl:R-EU_0207/2V -> rcl:R-EU_0204/7
- R22: device rcl:R-EU_0204/7 -> rcl:R-EU_0207/2V
Connections:
- removed net N$1: D1.A, R2.2
- removed net N$36: IC2A.OUT
- removed net N$4: IC2A.+IN, R6.2, R7.1
- removed net N$7: D2.A, R6.1
- removed net N$8: R7.2, R8.S
- new net 12V-MEASURE: IC2A.-IN, IC2A.OUT
- new net CPURX: MODUL1.D0/RX, VCC_GND_TX_RX.3
- new net CPUTX: MODUL1.D1/TX, VCC_GND_TX_RX.4
- net +12V: now also R2.2
- net +5V: now also SV1.1, VCC_GND_TX_RX.1; no longer +5V.P, R1.1, R8.E
- net GND: now also R1.1, SV1.3, VCC_GND_TX_RX.2; no longer D2.C, GND.P
- net M+: no longer D1.C
- net N$17: now also SV1.2; no longer HALSENSOR.P
- net N$2: now also IC2A.+IN; no longer IC2A.-IN
Other:
- note removed: "MOSFET current sens"
- moved on the sheet: B+, B-, IC2A, R1, R2
